Commit message: modified:   description/robot_core2.xacro

File: description/robot_core2.xacro (robot description, xacro)
@@ -35,13 +35,11 @@
             <material name="white"/>
         </visual>
-        <!-- <collision>
+        <collision>
             <origin xyz="0.2575 0 0.0675"/>
             <geometry>
-                <box size="0.515 0.31 0.135"/>
+                <box size="0.515 0.31 0.097"/>
+                <!-- l b h -->
             </geometry>
         </collision>
-        <xacro:inertial_box mass="0.5" x="0.515" y="0.31" z="0.135">
-            <origin xyz="0.2575 0 0.0675" rpy="0 0 0"/>
-        </xacro:inertial_box>   -->
     </link>
     <!-- <gazebo reference="chassis">
@@ -98,5 +96,5 @@
 </link>
 <!-- FRONT -->
-<joint name="front_wheel_steer_joint" type="revolute">
+<!-- <joint name="front_wheel_steer_joint" type="revolute">
     <limit lower="-1" upper="1" effort="1" velocity="5"/>
     <axis xyz="0 0 1"/>
@@ -112,8 +110,8 @@
       <material name="black"/>
     </visual>
-  </link>
+  </link>  -->
   <!-- FRONT LEFT WHEEL -->
 <joint name="front_left_wheel_joint" type="continuous">
-    <parent link="front_wheel_steer"/>
+    <parent link="front_left_wheel_steer"/>
     <child link="front_left_wheel"/>
     <origin xyz="0 0.18 0.0194" rpy="-${pi/2} 0 0"/>
@@ -130,7 +128,22 @@
     </visual>
 </link>
+<joint name="front_left_wheel_steer_joint" type="revolute">
+    <limit lower="-1" upper="1" effort="1" velocity="5"/>
+    <axis xyz="0 0 1"/>
+    <parent link="base_link"/>
+    <child link="front_left_wheel_steer"/>
+    <origin rpy="0 0 0" xyz="0.360 0 0"/>
+  </joint>
+<link name="front_left_wheel_steer">
+    <visual>
+      <geometry>
+        <cylinder length="0.01" radius="0.01"/>
+      </geometry>
+      <material name="black"/>
+    </visual>
+  </link>
   <!-- FRONT RIGHT WHEEL -->
 <joint name="front_right_wheel_joint" type="continuous">
-    <parent link="front_wheel_steer"/>
+    <parent link="front_right_wheel_steer"/>
     <child link="front_right_wheel"/>
     <origin xyz="0 -0.18 0.0194" rpy="-${pi/2} 0 0"/>
@@ -147,3 +160,18 @@
     </visual>
 </link>
+<joint name="front_right_wheel_steer_joint" type="revolute">
+    <limit lower="-1" upper="1" effort="1" velocity="5"/>
+    <axis xyz="0 0 1"/>
+    <parent link="base_link"/>
+    <child link="front_right_wheel_steer"/>
+    <origin rpy="0 0 0" xyz="0.360 0 0"/>
+  </joint>
+<link name="front_right_wheel_steer">
+    <visual>
+      <geometry>
+        <cylinder length="0.01" radius="0.01"/>
+      </geometry>
+      <material name="black"/>
+    </visual>
+  </link>
     </robot>

Commit message: modified:   description/robot_core2.xacro

File: description/robot_core2.xacro (robot description, xacro)
@@ -1,5 +1,5 @@
 <?xml version="1.0"?>
 <robot xmlns:xacro="http://www.ros.org/wiki/xacro" >
-    <!-- <xacro:include filename="inertial_macros.xacro"/> -->
+    <xacro:include filename="inertial_macros.xacro"/>
     <material name="white">
         <color rgba="1 1 1 1" />
@@ -42,8 +42,11 @@
             </geometry>
         </collision>
+        <xacro:inertial_box mass="0.5" x="0.515" y="0.31" z="0.097">
+            <origin xyz="0.2575 0 0.0675" rpy="0 0 0"/>
+        </xacro:inertial_box>
     </link>
-    <!-- <gazebo reference="chassis">
+    <gazebo reference="chassis">
         <material>Gazebo/White</material>
-    </gazebo> -->
+    </gazebo>
     <!-- UPPER CHASSIS LINK -->
 <joint name="upper_chassis_joint" type="fixed">
@@ -60,5 +63,17 @@
         <material name="red"/>
     </visual>
-</link>
+    <collision>
+        <origin xyz="0 0 0.038" rpy="0 0 0"/>
+        <geometry>
+            <box size="0.263 0.31 0.04"/>
+        </geometry>
+    </collision>
+        <xacro:inertial_box mass="0.5" x="0.263" y="0.31" z="0.04">
+            <origin xyz="0 0 0.038" rpy="0 0 0"/>
+        </xacro:inertial_box>
+</link>
+    <gazebo reference="upper_chassis">
+        <material>Gazebo/Red</material>
+    </gazebo>
   <!-- Rear LEFT WHEEL -->
 <joint name="rear_left_wheel_joint" type="continuous">
@@ -70,4 +85,5 @@
     <axis xyz="0 0 1"/>
 </joint>
+<!--  -->
 <link name="rear_left_wheel">
     <visual>
@@ -77,5 +93,19 @@
         <material name="blue"/>
     </visual>
-</link>
+<!--  -->
+    <collision>
+        <geometry>
+            <cylinder length="0.04" radius="0.0485" />
+        </geometry>
+    </collision>
+<!--  -->
+    <xacro:inertial_cylinder mass="0.1" length="0.04" radius="0.0485">
+            <origin xyz="0 0 0" rpy="0 0 0"/>
+        </xacro:inertial_cylinder>
+</link>
+<!--  -->
+    <gazebo reference="rear_left_wheel">
+        <material>Gazebo/Blue</material>
+    </gazebo>
   <!-- Rear RIGHT WHEEL -->
 <joint name="rear_right_wheel_joint" type="continuous">
@@ -87,4 +117,5 @@
     <axis xyz="0 0 -1"/>
 </joint>
+<!--  -->
 <link name="rear_right_wheel">
     <visual>
@@ -94,5 +125,18 @@
         <material name="blue"/>
     </visual>
-</link>
+<!--  -->
+    <collision>
+        <geometry>
+            <cylinder length="0.04" radius="0.0485" />
+        </geometry>
+    </collision>
+<!--  -->
+        <xacro:inertial_cylinder mass="0.1" length="0.04" radius="0.0485">
+            <origin xyz="0 0 0" rpy="0 0 0"/>
+        </xacro:inertial_cylinder>
+</link>
+    <gazebo reference="rear_right_wheel">
+        <material>Gazebo/Blue</material>
+    </gazebo>
 <!-- FRONT -->
 <!-- <joint name="front_wheel_steer_joint" type="revolute">
@@ -113,11 +157,12 @@
   <!-- FRONT LEFT WHEEL -->
 <joint name="front_left_wheel_joint" type="continuous">
-    <parent link="front_left_wheel_steer"/>
+    <parent link="base_link"/>
     <child link="front_left_wheel"/>
-    <origin xyz="0 0.18 0.0194" rpy="-${pi/2} 0 0"/>
+    <origin xyz="0.360 0.18 0.0194" rpy="-${pi/2} 0 0"/>
     <!-- y = b + thickness of wheel/2 + 0.5(mm) -->
     <!-- connected with base link -->
     <axis xyz="0 0 1"/>
 </joint>
+<!--  -->
 <link name="front_left_wheel">
     <visual>
@@ -127,29 +172,30 @@
         <material name="blue"/>
     </visual>
-</link>
-<joint name="front_left_wheel_steer_joint" type="revolute">
-    <limit lower="-1" upper="1" effort="1" velocity="5"/>
-    <axis xyz="0 0 1"/>
-    <parent link="base_link"/>
-    <child link="front_left_wheel_steer"/>
-    <origin rpy="0 0 0" xyz="0.360 0 0"/>
-  </joint>
-<link name="front_left_wheel_steer">
-    <visual>
-      <geometry>
-        <cylinder length="0.01" radius="0.01"/>
-      </geometry>
-      <material name="black"/>
-    </visual>
-  </link>
+<!--  -->
+    <collision>
+        <geometry>
+            <cylinder length="0.04" radius="0.0485" />
+        </geometry>
+    </collision>
+<!--  -->
+    <xacro:inertial_cylinder mass="0.1" length="0.04" radius="0.0485">
+            <origin xyz="0 0 0" rpy="0 0 0"/>
+    </xacro:inertial_cylinder>
+</link>
+<!--  -->
+    <gazebo reference="left_wheel">
+        <material>Gazebo/Blue</material>
+    </gazebo>
+<!--  -->
   <!-- FRONT RIGHT WHEEL -->
 <joint name="front_right_wheel_joint" type="continuous">
-    <parent link="front_right_wheel_steer"/>
+    <parent link="base_link"/>
     <child link="front_right_wheel"/>
-    <origin xyz="0 -0.18 0.0194" rpy="-${pi/2} 0 0"/>
+    <origin xyz="0.360 -0.18 0.0194" rpy="-${pi/2} 0 0"/>
     <!-- y = b + thickness of wheel/2 + 0.5(mm) -->
     <!-- connected with base link -->
     <axis xyz="0 0 -1"/>
 </joint>
+<!--  -->
 <link name="front_right_wheel">
     <visual>
@@ -159,19 +205,18 @@
         <material name="blue"/>
     </visual>
-</link>
-<joint name="front_right_wheel_steer_joint" type="revolute">
-    <limit lower="-1" upper="1" effort="1" velocity="5"/>
-    <axis xyz="0 0 1"/>
-    <parent link="base_link"/>
-    <child link="front_right_wheel_steer"/>
-    <origin rpy="0 0 0" xyz="0.360 0 0"/>
-  </joint>
-<link name="front_right_wheel_steer">
-    <visual>
-      <geometry>
-        <cylinder length="0.01" radius="0.01"/>
-      </geometry>
-      <material name="black"/>
-    </visual>
-  </link>
+<!--  -->
+    <collision>
+        <geometry>
+            <cylinder length="0.04" radius="0.0485" />
+        </geometry>
+    </collision>
+<!--  -->
+    <xacro:inertial_cylinder mass="0.1" length="0.04" radius="0.0485">
+            <origin xyz="0 0 0" rpy="0 0 0"/>
+    </xacro:inertial_cylinder>
+</link>
+<!--  -->
+    <gazebo reference="front_right_wheel">
+        <material>Gazebo/Blue</material>
+    </gazebo>
     </robot>
